Commit message: fixed minor eror in d3out calculation and a small mislaignment in urdf

File: scarabot_description/urdf/scarabot.urdf (robot description, URDF)
Before this commit: robot SCARA, 7 links, 6 joints
Joints:
- joint joint_6: origin xyz=1       0      -0.6 rpy=0  0  0 -> xyz=1       0      -0.5 rpy=0  0  0
